File: PCB_Wristband/Blind_Assistance_EE_Project.kicad_sch (KiCad schematic)
At the start: 30 parts, among them J1 BT1, J2 USB_C_Receptacle_PowerOnly_6P, M1 Motor_DC, M2 Motor_DC, M3 Motor_DC, Q2 AO3400A, Q3 AO3400A, Q4 AO3400A, U1 TP4056-42-ESOP8, U2 BNO055, U3 ESP32-C3_SUPERMINI_TH

Commit message: updated and replaced parts with newer ones for schematic.
Parts:
- added M5, M7, M9: Motor_AC, symbol Motor:Motor_AC
- added SW1, SW2: PTS526_SM15_SMTR2_LFS, PTS526_SM15_SMTR2_LFS:PTS526SM15SMTR2LFS, symbol New_Library2:PTS526_SM15_SMTR2_LFS
- added U12, U13: TCA9548ARGER, Package_DFN_QFN:Texas_RGE0024C_VQFN-24-1EP_4x4mm_P0.5mm_EP2.1x2.1mm, symbol Interface_Expansion:TCA9548ARGER
- added U4: ESP32-S3-SuperMini, ESP32-S3-SuperMini:ESP32-S3-SuperMini, symbol New_Library2:ESP32-S3-SuperMini
- added U5: BNO055, Package_LGA:LGA-28_5.2x3.8mm_P0.5mm, symbol Sensor_Motion:BNO055
- added U6, U7, U8: DRV2605LDGS, Package_SO:TSSOP-10_3x3mm_P0.5mm, symbol Driver:DRV2605LDGS
Connections:
- new net: SW1.1, SW1.2
- new net: SW1.3, SW1.4
- new net: SW2.1, SW2.2
- new net: SW2.3, SW2.4
Other:
- moved on the sheet: C1, C2, C3, C4, C5, C6, C7, D1, D2, D3, J1, J2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

Commit message: Motors and haptics connected (To Do: connect VDD of driver to 3.3V source)
Parts:
- added C10, C9: C, symbol Device:C
- added C11, C12, C14, C15, C16: 1uF, symbol Device:C
- added C13, C8: 1uF, Package_SON:Texas_DSG0008A_WSON-8-1EP_2x2mm_P0.5mm_EP0.9x1.6mm, symbol Device:C
- added M10, M6, M8: Motor_AC, symbol Motor:Motor_AC
- added U10, U11, U9: DRV2605LDGS, Package_SO:TSSOP-10_3x3mm_P0.5mm, symbol Driver:DRV2605LDGS
- added U14: ESP32-S3-SuperMini, ESP32-S3-SuperMini:ESP32-S3-SuperMini, symbol New_Library2:ESP32-S3-SuperMini
Connections:
- net +3V3: now also U4.3 (3V3), U6.10 (VDD), U7.10 (VDD), U8.10 (VDD)
- net GND: now also U4.2 (GND), U6.4 (IN/TRIG), U6.8 (GND), U7.4 (IN/TRIG), U7.8 (GND), U8.4 (IN/TRIG), U8.8 (GND), C10.2, C11.2, C12.2, C13.2, C8.2, C9.2, U10.4 (IN/TRIG), U10.8 (GND), U11.4 (IN/TRIG), U11.8 (GND), U9.4 (IN/TRIG), U9.8 (GND)
- net at U6.1 (REG): now also C10.1
- net at U6.2 (SCL): now also U4.9 (GPIO_8), U7.2 (SCL), U8.2 (SCL)
- net at U6.3 (SDA): now also U4.8 (GPIO_9), U7.3 (SDA), U8.3 (SDA)
- net at U6.5 (EN): now also U4.16 (GPIO_1)
- net at U6.7 (OUT+): now also M5.1
- net at U6.9 (OUT-): now also M5.2
- net at U8.1 (REG): now also C8.1
- net at U8.5 (EN): now also U4.14 (GPIO_3)
- net at U8.7 (OUT+): now also M9.1
- net at U8.9 (OUT-): now also M9.2
- net at U7.1 (REG): now also C9.1
- net at U7.5 (EN): now also U4.15 (GPIO_2)
- net at U7.7 (OUT+): now also M7.1
- net at U7.9 (OUT-): now also M7.2
- new net: U11.5 (EN), U14.10 (GPIO_7)
- new net: U10.5 (EN), U14.11 (GPIO_6)
- new net: U14.12 (GPIO_5), U9.5 (EN)
- new net: U10.3 (SDA), U11.3 (SDA), U14.6 (GPIO_11), U9.3 (SDA)
- new net: U10.2 (SCL), U11.2 (SCL), U14.7 (GPIO_10), U9.2 (SCL)
- new net: M6.1, U9.7 (OUT+)
- new net: M6.2, U9.9 (OUT-)
- new net: C16.1, U11.10 (VDD)
- new net: C11.1, U9.1 (REG)
- new net: C14.1, U9.10 (VDD)
- new net: C12.1, U10.1 (REG)
- new net: C13.1, U11.1 (REG)
- new net: M10.1, U11.7 (OUT+)
- new net: M10.2, U11.9 (OUT-)
- new net: C15.1, U10.10 (VDD)
- new net: M8.1, U10.7 (OUT+)
- new net: M8.2, U10.9 (OUT-)
- no-connect marks 12 -> 21
Other:
- moved on the sheet: M5, M7, M9, SW1, SW2, U4, U5, U6, U7, U8
